File: Eagle/Helmet_Drop_V1.brd (EAGLE design)
At the start: 172.7 x 106.4 mm, 25 parts, among them Q3 MOSFET-NCH, Q4 MOSFET-NCH, Q5 MOSFET-NCH, U1 ITSYBITSY_5V

Commit message: Updated to make newest repository location
Connections:
- new net N$5: U1.D7, U1.RES
Routing:
- net N$5: track 0.00 -> 26.6 mm
Changed lines of the file:
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@@
 <drawing>
 <settings>
-<setting alwaysvectorfont="yes"/>
+<setting alwaysvectorfont="no"/>
 <setting keepoldvectorfont="yes"/>
 <setting verticaltext="up"/>
@@
 <contactref element="AUXILLARY_LIGHTS" pad="3"/>
 </signal>
+<signal name="N$5">
+<contactref element="U1" pad="D7"/>
+<contactref element="U1" pad="RES"/>
+<wire x1="86.4108" y1="32.2326" x2="86.4108" y2="32.9184" width="0.254" layer="16"/>
+<wire x1="100.1268" y1="18.5166" x2="86.4108" y2="32.2326" width="0.254" layer="16"/>
+<wire x1="100.1268" y1="14.1732" x2="100.1268" y2="18.5166" width="0.254" layer="16"/>
+<wire x1="101.6" y1="12.7" x2="100.1268" y2="14.1732" width="0.254" layer="16"/>
+<wire x1="86.4108" y1="32.9184" x2="86.36" y2="33.02" width="0.254" layer="16"/>
+</signal>
 </signals>
