File: Eagle/Helmet_Drop_V1.sch (EAGLE design)
At the start: 25 parts, among them Q3 MOSFET-NCH, Q4 MOSFET-NCH, Q5 MOSFET-NCH, U1 ITSYBITSY_5V

Commit message: Updated to make newest repository location
Connections:
- new net N$5: U1.D7, U1.RST
Changed lines of the file:
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@@
+</segment>
+</net>
+<net name="N$5" class="0">
+<segment>
+<pinref part="U1" gate="G$1" pin="D7"/>
+<wire x1="114.3" y1="142.24" x2="132.08" y2="142.24" width="0.1524" layer="91"/>
+<wire x1="132.08" y1="142.24" x2="132.08" y2="170.18" width="0.1524" layer="91"/>
+<wire x1="132.08" y1="170.18" x2="78.74" y2="170.18" width="0.1524" layer="91"/>
+<pinref part="U1" gate="G$1" pin="RST"/>
+<wire x1="78.74" y1="170.18" x2="78.74" y2="162.56" width="0.1524" layer="91"/>
+<wire x1="78.74" y1="162.56" x2="81.28" y2="162.56" width="0.1524" layer="91"/>
 </segment>
 </net>
