File: Eagle/Helmet_Drop_V2.1.brd (EAGLE design)
At the start: 106.4 x 172.7 mm, 30 parts, among them Q3 MOSFET-NCH, Q4 MOSFET-NCH, Q5 MOSFET-NCH, U1 TH_DS_LIBRARIES_ITSYBITSY_5V, X1 MSTBA4, X2 TH_DS_LIBRARIES_MSTBA4

Commit message: board fix
Connections:
- removed net VCC: JMP3.1, JP2.1
- net 5V: now also JMP3.1, JP2.1
Routing:
- net 5V: track 265.7 -> 306.6 mm
- net VCC: track 12.1 -> 0.00 mm
Other:
- board text added: "Only Jump Data Pins OR Ground Pins DO NOT CONNECT BOTH Default should be DATA"
- board text removed: "Only Jump Data Pins OR Ground Pins DO NOT CONNECT BOTH"
Changed lines of the file:
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@@
 <text x="66.167" y="115.824" size="1.778" layer="25" rot="R180">GND</text>
 <text x="59.817" y="115.824" size="1.778" layer="25" rot="R180">GND</text>
-<text x="49.53" y="105.41" size="1.778" layer="25">Only Jump Data Pins
+<text x="49.53" y="101.6" size="1.778" layer="25">Only Jump Data Pins
 OR Ground Pins
-DO NOT CONNECT BOTH</text>
+DO NOT CONNECT BOTH
+Default should be DATA</text>
 <text x="19.05" y="31.75" size="1.778" layer="25" rot="R180">12V</text>
 <text x="102.362" y="77.978" size="2.1844" layer="25" rot="R180">24V</text>
@@
 <wire x1="111.8616" y1="60.6552" x2="111.76" y2="60.96" width="0.635" layer="16"/>
 <wire x1="23.1648" y1="38.608" x2="22.86" y2="38.5064" width="0.635" layer="16"/>
+<contactref element="JP2" pad="1"/>
+<contactref element="JMP3" pad="1"/>
+<wire x1="76.708" y1="127.8128" x2="76.708" y2="133.2992" width="0.635" layer="1"/>
+<wire x1="81.28" y1="123.2408" x2="76.708" y2="127.8128" width="0.635" layer="1"/>
+<wire x1="76.708" y1="133.2992" x2="76.63" y2="133.35" width="0.635" layer="1"/>
+<wire x1="81.28" y1="123.2408" x2="81.28" y2="123.19" width="0.635" layer="1"/>
+<wire x1="97.4344" y1="123.2408" x2="81.28" y2="123.2408" width="0.635" layer="16"/>
+<wire x1="106.172" y1="131.9784" x2="97.4344" y2="123.2408" width="0.635" layer="16"/>
+<wire x1="81.28" y1="123.2408" x2="81.28" y2="123.19" width="0.635" layer="16"/>
+<wire x1="106.172" y1="131.9784" x2="106.426" y2="132.08" width="0.635" layer="16"/>
 </signal>
 <signal name="D0" class="2">
@@
 <wire x1="106.4768" y1="121.92" x2="106.426" y2="121.92" width="0.254" layer="16"/>
 </signal>
-<signal name="VCC" class="1">
-<contactref element="JP2" pad="1"/>
-<contactref element="JMP3" pad="1"/>
-<wire x1="76.708" y1="127.8128" x2="76.708" y2="133.2992" width="0.635" layer="1"/>
-<wire x1="81.28" y1="123.2408" x2="76.708" y2="127.8128" width="0.635" layer="1"/>
-<wire x1="76.708" y1="133.2992" x2="76.63" y2="133.35" width="0.635" layer="1"/>
-<wire x1="81.28" y1="123.2408" x2="81.28" y2="123.19" width="0.635" layer="1"/>
-</signal>
 <signal name="EN" class="2">
