File: Eagle/Helmet_Drop_V2.0.sch (EAGLE design)
At the start: 27 parts, among them Q3 MOSFET-NCH, Q4 MOSFET-NCH, Q5 MOSFET-NCH, U1 TH_DS_LIBRARIES_ITSYBITSY_5V, X1 MSTBA4

Commit message: Moved connectors for ease of access
Parts:
- removed 5V_IN, SDA_SCL: MSTBA2, th_libraries:MSTBA2
- added JMP3: 0R-JUMPA, jump-0r-smd:0R-JUMPA
- added JP2: (no value), microbuilder:HEADER-1X570MIL
- added U$19, U$21: MOUNTINGHOLE2.5, microbuilder:MOUNTINGHOLE2.5
- added X2: TH_DS_LIBRARIES_MSTBA4, OMSI_Default_V1:TH_DS_LIBRARIES_MSTBA4
Connections:
- removed net D2: SDA_SCL-1.1, U1.SDA/D2
- removed net D3: SDA_SCL-2.1, U1.SCL/D3
- new net EN: JMP3-0R.2, JP2.5
- new net SCL: JP2.3, U1.SCL/D3, X2-2.1
- new net SDA: JP2.4, U1.SDA/D2, X2-1.1
- new net VCC: JMP3-0R.1, JP2.1
- net 5V: now also X2-3.1; no longer 5V_IN-1.1
- net GND: now also JMP3-0R.3, JP2.2, X2-4.1; no longer 5V_IN-2.1
Other:
- note added: "I2C Pullups & Shift"
- note added: "ON LED"
- note added: "Power supply"
- note added: "STEMMA/I2C Headers"

Commit message: update
Parts:
- added X3: PHOENIX_508_2PIN, OMSI_Default_V1:PHOENIX_508_2PIN
- U1: value TH_DS_LIBRARIES_ITSYBITSY_5V -> ADAFRUIT_ITSYBITSY_5V; device Helmet_Drop_V1.5:TH_DS_LIBRARIES_ITSYBITSY_5V -> OMSI_Default_V1:ADAFRUIT_ITSYBITSY_5V
Connections:
- new net N$2: U1.D13, X3-2.1
- net D0: now also U1.RX; no longer U1.RX/D0
- net D1: now also U1.TX; no longer U1.TX/D1
- net GND: now also X3-1.1
- net SCL: now also U1.SCL; no longer U1.SCL/D3
- net SDA: now also U1.SDA; no longer U1.SDA/D2
