File: Eagle/Helmet_Drop_V2.1.sch (EAGLE design)
At the start: 30 parts, among them Q3 MOSFET-NCH, Q4 MOSFET-NCH, Q5 MOSFET-NCH, U1 TH_DS_LIBRARIES_ITSYBITSY_5V, X1 MSTBA4, X2 TH_DS_LIBRARIES_MSTBA4

Commit message: updated indicator lights
Parts:
- added D1, D2: (no value), SparkFun-LED:LED1206
- added Q1, Q2: 2.5A/30V/105mΩ, SparkFun-DiscreteSemi:MOSFET_PCH-DMG2307L
- added R1, R3: 10k, SparkFun-Passives:RESISTOR0805-RES
- added R2, R4: 1000, SparkFun-Passives:RESISTOR0805-RES
Connections:
- removed net D0: U1.RX/D0, X1-4.1
- removed net D4: REED_IN-3.1, U1.D4
- new net N$2: Q2.D, R2.1
- new net N$3: Q1.D, R4.1
- new net N$4: D2.A, R4.2
- new net N$5: D1.A, R2.2
- new net REEDIN: Q2.G, R1.2, REED_IN-3.1, U1.D4
- new net SAFETYSWITCH: Q1.G, R3.2, U1.RX/D0, X1-4.1
- net 5V: now also Q1.S, Q2.S, R1.1, R3.1
- net GND: now also D1.C, D2.C
Other:
- note added: "Button Indicator"
- note added: "To Switch"
- note added: "To input"
- moved on the sheet: 10K2, 10K3, Q3, Q4

Commit message: cleanup
Parts:
- removed JP2: (no value), microbuilder:HEADER-1X570MIL
- removed S10, S11, S12, S5, S7, S9: STANDOFF_ELECTRICAL5-32, th_libraries:STANDOFF_ELECTRICAL5-32
- removed U$19, U$21: MOUNTINGHOLE2.5, microbuilder:MOUNTINGHOLE2.5
- added S1, S2, S3, S4, S6, S8: GND_HOLE, OMSI_Default_V1:GND_HOLE
- added TP3, TP4: TEST_POINTTP_15TH_THRU, OMSI_Default_V1:TEST_POINTTP_15TH_THRU
- added U$1: I2C_EXTENDER, OMSI_Default_V1:I2C_EXTENDER
- 10K2, 10K3, 10K4: device adafruit:R-US_M0805 -> OMSI_Default_V1:RESISTORS0805-RES
- 12V_IN, IR_IN, REED_IN: value MSTBA3 -> PHOENIX_508_3PIN; device con-phoenix-508:MSTBA3 -> OMSI_Default_V1:PHOENIX_508_3PIN
- 24V: value MSTBA2 -> PHOENIX_508_2PIN; device th_libraries:MSTBA2 -> OMSI_Default_V1:PHOENIX_508_2PIN
- AUXILLARY_LIGHTS1, STEPPER_MOTOR: value MSTBA6 -> PHOENIX_508_6PIN; device con-phoenix-508:MSTBA6 -> OMSI_Default_V1:PHOENIX_508_6PIN
- D1, D2: device SparkFun-LED:LED1206 -> OMSI_Default_V1:GENERIC_LED1206
- JMP1, JMP2: value 0R-JUMPB -> SMD_JUMPERA; device jump-0r-smd:0R-JUMPB -> OMSI_Default_V1:SMD_JUMPERA
- JMP3: value 0R-JUMPA -> SMD_JUMPERA; device jump-0r-smd:0R-JUMPA -> OMSI_Default_V1:SMD_JUMPERA
- LOCK_LIGHTS: value MSTBA4 -> PHOENIX_508_4PIN; device th_libraries:MSTBA4 -> OMSI_Default_V1:PHOENIX_508_4PIN
- Q1, Q2: value 2.5A/30V/105mΩ -> MOSFET-PCHIRLML9301TRPBF; device SparkFun-DiscreteSemi:MOSFET_PCH-DMG2307L -> OMSI_Default_V1:MOSFET-PCHIRLML9301TRPBF
- Q3, Q4, Q5: value MOSFET-NCH -> 310mA/60V/1.6Ω; device th_ds_libraries:MOSFET-NCH -> OMSI_Default_V1:MOSFET-NCH
- R1, R2, R3, R4: device SparkFun-Passives:RESISTOR0805-RES -> OMSI_Default_V1:RESISTORS0805-RES
- TP1, TP2: value PTR2 -> TEST_POINTTP_15TH_THRU; device testpad:PTR2 -> OMSI_Default_V1:TEST_POINTTP_15TH_THRU
- U1: value TH_DS_LIBRARIES_ITSYBITSY_5V -> ADAFRUIT_ITSYBITSY_5V; device Helmet_Drop_V1.5:TH_DS_LIBRARIES_ITSYBITSY_5V -> OMSI_Default_V1:ADAFRUIT_ITSYBITSY_5V
- X1: value MSTBA4 -> PHOENIX_508_4PIN; device con-phoenix-508:MSTBA4 -> OMSI_Default_V1:PHOENIX_508_4PIN
- X2: value TH_DS_LIBRARIES_MSTBA4 -> PHOENIX_508_4PIN; device OMSI_Default_V1:TH_DS_LIBRARIES_MSTBA4 -> OMSI_Default_V1:PHOENIX_508_4PIN
Connections:
- net 12V: now also TP4.1; no longer TP2-2.TP
- net 24V: now also TP1.1; no longer TP1-1.TP
- net 5V: now also JMP3.1, TP3.1, U$1.5; no longer JMP3-0R.1, JP2.1, TP2-1.TP
- net D1: now also U1.TX; no longer U1.TX/D1
- net D5: now also JMP1.1; no longer JMP1-0R.3
- net D5J: now also JMP1.2; no longer JMP1-0R.2
- net D7: now also JMP2.1; no longer JMP2-0R.3
- net D7J: now also JMP2.2; no longer JMP2-0R.2
- net EN: now also JMP3.2, U$1.1; no longer JMP3-0R.2, JP2.5
- net GND: now also JMP1.3, JMP2.3, JMP3.3, S1.P$1, S2.P$1, S3.P$1, S4.P$1, S6.P$1, S8.P$1, TP2.1, U$1.4; no longer JMP1-0R.1, JMP2-0R.1, JMP3-0R.3, JP2.2, S10.P$1, S11.P$1, S12.P$1, S5.P$1, S7.P$1, S9.P$1, TP1-2.TP
- net SAFETYSWITCH: now also U1.RX; no longer U1.RX/D0
- net SCL: now also U$1.3, U1.SCL; no longer JP2.3, U1.SCL/D3
- net SDA: now also U$1.2, U1.SDA; no longer JP2.4, U1.SDA/D2
Other:
- note removed: "Button Indicator"
- note removed: "I2C Pullups & Shift"
- note removed: "ON LED"
- note removed: "Power supply"
- note removed: "STEMMA/I2C Headers"
